Commit message: Tune Gazebo caster contact and diff-drive control mapping

File: src/yaseen_differential_robot/urdf/robot_description.xacro (robot description, xacro)
@@ -1,331 +1,320 @@
 <?xml version="1.0"?>
 <robot xmlns:xacro="http://www.ros.org/wiki/xacro">
-<xacro:macro name="yaseen_description">
-  <link name="base_footprint"/>
-  <link
-    name="base_link">
-    <inertial>
-      <origin
-        xyz="-0.0246664991701579 5.70622526084585E-06 -0.065175547408044"
+  <xacro:macro name="yaseen_description">
+    <link name="base_footprint"/>
+    <link name="base_link">
+      <inertial>
+        <origin
+          xyz="-0.0246664991701579 5.70622526084585E-06 -0.065175547408044"
+          rpy="0 0 0" />
+        <mass
+          value="11.8117325473893" />
+        <inertia
+          ixx="0.130576626113656"
+          ixy="1.47971062390579E-07"
+          ixz="0.00285071032522239"
+          iyy="0.168919301848653"
+          iyz="1.07757011014447E-08"
+          izz="0.0962622389900477" />
+      </inertial>
+      <visual>
+        <origin
+          xyz="0 0 0"
+          rpy="0 0 0" />
+        <geometry>
+          <mesh
+            filename="package://yaseen_differential_robot/meshes/base_link.STL" />
+        </geometry>
+        <material
+          name="">
+          <color
+            rgba="0.498039215686275 0.498039215686275 0.498039215686275 1" />
+        </material>
+      </visual>
+      <collision>
+        <origin
+          xyz="0 0 0.02"
+          rpy="0 0 0" />
+        <geometry>
+          <box size="0.55 0.35 0.08"/>
+        </geometry>
+      </collision>
+    </link>
+    <joint name="base_footprint_joint" type="fixed">
+      <origin
+        xyz="0 0 0.58365"
+        rpy="0 0 3.141592653589793" />
+      <parent
+        link="base_footprint" />
+      <child
+        link="base_link" />
+    </joint>
+    <link name="wheel_right_link">
+      <inertial>
+        <origin
+          xyz="-2.43019668694222E-06 1.85668461649691E-06 -0.0204728433099643"
+          rpy="0 0 0" />
+        <mass
+          value="0.516905713246417" />
+        <inertia
+          ixx="0.00125613924285597"
+          ixy="2.11747326433519E-09"
+          ixz="2.64299917067243E-08"
+          iyy="0.00125611448213454"
+          iyz="-1.32101831494911E-08"
+          izz="0.00238429646215864" />
+      </inertial>
+      <visual>
+        <origin
+          xyz="0 0 0"
+          rpy="0 0 0" />
+        <geometry>
+          <mesh
+            filename="package://yaseen_differential_robot/meshes/wheel_right_link.STL" />
+        </geometry>
+        <material
+          name="">
+          <color
+            rgba="0.792156862745098 0.819607843137255 0.933333333333333 1" />
+        </material>
+      </visual>
+      <collision>
+        <origin
+          xyz="0 0 0"
+          rpy="0 0 0" />
+        <geometry>
+          <cylinder radius="0.0855" length="0.033"/>
+        </geometry>
+      </collision>
+    </link>
+    <joint
+      name="wheel_right_joint"
+      type="continuous">
+      <origin
+        xyz="-0.33125 -0.25295 -0.49815"
+        rpy="-1.5708 0 3.1416" />
+      <parent
+        link="base_link" />
+      <child
+        link="wheel_right_link" />
+      <axis
+        xyz="0 0 -1" />
+      <dynamics
+        damping="0.1"
+        friction="0.1" />
+    </joint>
+    <link name="wheel_left_link">
+      <inertial>
+        <origin
+          xyz="3.05776156006576E-06 -3.77816526953012E-08 -0.0204728432555836"
+          rpy="0 0 0" />
+        <mass
+          value="0.516905716540766" />
+        <inertia
+          ixx="0.00125612706197731"
+          ixy="1.24388995856856E-08"
+          ixz="-2.91071422970173E-08"
+          iyy="0.00125612402313693"
+          iyz="-5.16913670862521E-09"
+          izz="0.00238429647597481" />
+      </inertial>
+      <visual>
+        <origin
+          xyz="0 0 0"
+          rpy="0 0 0" />
+        <geometry>
+          <mesh
+            filename="package://yaseen_differential_robot/meshes/wheel_left_link.STL" />
+        </geometry>
+        <material
+          name="">
+          <color
+            rgba="0.792156862745098 0.819607843137255 0.933333333333333 1" />
+        </material>
+      </visual>
+      <collision>
+        <origin
+          xyz="0 0 0"
+          rpy="0 0 0" />
+        <geometry>
+          <cylinder radius="0.0855" length="0.033"/>
+        </geometry>
+      </collision>
+    </link>
+    <joint
+      name="wheel_left_joint"
+      type="continuous">
+      <origin
+        xyz="-0.33125 0.25345 -0.49815"
+        rpy="1.5708 0 3.1416" />
+      <parent
+        link="base_link" />
+      <child
+        link="wheel_left_link" />
+      <axis
+        xyz="0 0 -1" />
+      <dynamics
+        damping="0.1"
+        friction="0.1" />
+    </joint>
+    <link name="caster_left_wheel_link">
+      <inertial>
+        <origin
+          xyz="-0.00849270707917538 0.0122148476204665 9.91213475813879E-05"
+          rpy="0 0 0" />
+        <mass
+          value="0.16436862013948" />
+        <inertia
+          ixx="0.000134032984026512"
+          ixy="4.88470723909831E-05"
+          ixz="-3.22329844113555E-08"
+          iyy="0.000114249682482447"
+          iyz="4.632156635282E-08"
+          izz="0.000205220433201827" />
+      </inertial>
+      <visual>
+        <origin
+          xyz="0 0 0"
+          rpy="0 0 0" />
+        <geometry>
+          <mesh
+            filename="package://yaseen_differential_robot/meshes/caster_left_wheel_link.STL" />
+        </geometry>
+        <material
+          name="">
+          <color
+            rgba="0.792156862745098 0.819607843137255 0.933333333333333 1" />
+        </material>
+      </visual>
+      <collision>
+        <origin
+          xyz="0 0 0"
+          rpy="0 0 0" />
+        <geometry>
+          <sphere radius="0.0372"/>
+        </geometry>
+      </collision>
+    </link>
+    <joint
+      name="caster_left_wheel_joint"
+      type="fixed">
+      <origin
+        xyz="0.26586 0.085525 -0.53206"
+        rpy="1.5708 0 3.1416" />
+      <parent
+        link="base_link" />
+      <child
+        link="caster_left_wheel_link" />
+      <axis
+        xyz="0 0 0" />
+      <limit
+        lower="0"
+        upper="0"
+        effort="0"
+        velocity="0" />
+    </joint>
+    <link name="caster_wheel_right_link">
+      <inertial>
+        <origin
+          xyz="-0.00849270707917676 -0.0122148476204665 -9.91213475806524E-05"
+          rpy="0 0 0" />
+        <mass
+          value="0.16436862013948" />
+        <inertia
+          ixx="0.000134032984026512"
+          ixy="-4.88470723909831E-05"
+          ixz="3.22329844113684E-08"
+          iyy="0.000114249682482447"
+          iyz="4.63215663527944E-08"
+          izz="0.000205220433201827" />
+      </inertial>
+      <visual>
+        <origin
+          xyz="0 0 0"
+          rpy="0 0 0" />
+        <geometry>
+          <mesh
+            filename="package://yaseen_differential_robot/meshes/caster_wheel_right_link.STL" />
+        </geometry>
+        <material
+          name="">
+          <color
+            rgba="0.792156862745098 0.819607843137255 0.933333333333333 1" />
+        </material>
+      </visual>
+      <collision>
+        <origin
+          xyz="0 0 0"
+          rpy="0 0 0" />
+        <geometry>
+          <sphere radius="0.0372"/>
+        </geometry>
+      </collision>
+    </link>
+    <joint
+      name="caster_wheel_right_joint"
+      type="fixed">
+      <origin
+        xyz="0.26586 -0.085525 -0.53206"
+        rpy="-1.5708 0 3.1416" />
+      <parent
+        link="base_link" />
+      <child
+        link="caster_wheel_right_link" />
+      <axis
+        xyz="0 0 0" />
+    </joint>
+    <link name="lidar_link">
+      <inertial>
+        <origin
+          xyz="-0.000565454433324009 -1.49381448554266E-05 -0.021701451940591"
+          rpy="0 0 0" />
+        <mass
+          value="0.165382751635991" />
+        <inertia
+          ixx="7.88651836105335E-05"
+          ixy="4.84717640920677E-08"
+          ixz="2.18479443959808E-06"
+          iyy="7.51902914938722E-05"
+          iyz="2.88601572509174E-08"
+          izz="0.000109946753058707" />
+      </inertial>
+      <visual>
+        <origin
+          xyz="0 0 0"
+          rpy="0 0 0" />
+        <geometry>
+          <mesh
+            filename="package://yaseen_differential_robot/meshes/lidar_link.STL" />
+        </geometry>
+        <material
+          name="">
+          <color
+            rgba="0.752941176470588 0.752941176470588 0.752941176470588 0.4" />
+        </material>
+      </visual>
+      <collision>
+        <origin
+          xyz="0 0 0"
+          rpy="0 0 0" />
+        <geometry>
+          <mesh
+            filename="package://yaseen_differential_robot/meshes/lidar_link.STL" />
+        </geometry>
+      </collision>
+    </link>
+    <joint
+      name="lidar_joint"
+      type="fixed">
+      <origin
+        xyz="0.2775 -0.00045 -0.4169"
         rpy="0 0 0" />
-      <mass
-        value="11.8117325473893" />
-      <inertia
-        ixx="0.130576626113656"
-        ixy="1.47971062390579E-07"
-        ixz="0.00285071032522239"
-        iyy="0.168919301848653"
-        iyz="1.07757011014447E-08"
-        izz="0.0962622389900477" />
-    </inertial>
-    <visual>
-      <origin
-        xyz="0 0 0"
-        rpy="0 0 0" />
-      <geometry>
-        <mesh
-          filename="package://yaseen_differential_robot/meshes/base_link.STL" />
-      </geometry>
-      <material
-        name="">
-        <color
-          rgba="0.498039215686275 0.498039215686275 0.498039215686275 1" />
-      </material>
-    </visual>
-    <collision>
-      <origin
-        xyz="0 0 0"
-        rpy="0 0 0" />
-      <geometry>
-        <mesh
-          filename="package://yaseen_differential_robot/meshes/base_link.STL" />
-      </geometry>
-    </collision>
-  </link>
-  <joint name="base_footprint_joint" type="fixed">
-    <origin
-      xyz="0 0 0.56206"
-      rpy="0 0 3.141592653589793" />
-    <parent
-      link="base_footprint" />
-    <child
-      link="base_link" />
-  </joint>
-  <link
-    name="wheel_right_link">
-    <inertial>
-      <origin
-        xyz="-2.43019668694222E-06 1.85668461649691E-06 -0.0204728433099643"
-        rpy="0 0 0" />
-      <mass
-        value="0.516905713246417" />
-      <inertia
-        ixx="0.00125613924285597"
-        ixy="2.11747326433519E-09"
-        ixz="2.64299917067243E-08"
-        iyy="0.00125611448213454"
-        iyz="-1.32101831494911E-08"
-        izz="0.00238429646215864" />
-    </inertial>
-    <visual>
-      <origin
-        xyz="0 0 0"
-        rpy="0 0 0" />
-      <geometry>
-        <mesh
-          filename="package://yaseen_differential_robot/meshes/wheel_right_link.STL" />
-      </geometry>
-      <material
-        name="">
-        <color
-          rgba="0.792156862745098 0.819607843137255 0.933333333333333 1" />
-      </material>
-    </visual>
-    <collision>
-      <origin
-        xyz="0 0 0"
-        rpy="0 0 0" />
-      <geometry>
-        <mesh
-          filename="package://yaseen_differential_robot/meshes/wheel_right_link.STL" />
-      </geometry>
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
File: src/yaseen_differential_robot/urdf/robot_gazebo.xacro (robot description, xacro)
@@ -8,3 +8,29 @@
     </gazebo>
   </xacro:macro>
+  <!-- Wheel friction (drive wheels) - Moderate realistic values -->
+  <gazebo reference="wheel_left_link">
+    <mu1>1.0</mu1>
+    <mu2>1.0</mu2>
+    <kp>10000.0</kp>
+    <kd>1.0</kd>
+    <minDepth>0.001</minDepth>
+    <maxVel>1.0</maxVel>
+  </gazebo>
+  <gazebo reference="wheel_right_link">
+    <mu1>1.0</mu1>
+    <mu2>1.0</mu2>
+    <kp>10000.0</kp>
+    <kd>1.0</kd>
+    <minDepth>0.001</minDepth>
+    <maxVel>1.0</maxVel>
+  </gazebo>
+  <!-- Low friction casters - VERY low to not interfere -->
+  <gazebo reference="caster_left_wheel_link">
+    <mu1>0.0</mu1>
+    <mu2>0.0</mu2>
+  </gazebo>
+  <gazebo reference="caster_wheel_right_link">
+    <mu1>0.0</mu1>
+    <mu2>0.0</mu2>
+  </gazebo>
 </robot>

Commit message: new urdf added

File: src/yaseen_differential_robot/urdf/robot_description.xacro (robot description, xacro)
@@ -6,15 +6,15 @@
       <inertial>
         <origin
-          xyz="-0.0246664991701579 5.70622526084585E-06 -0.065175547408044"
-          rpy="0 0 0" />
-        <mass
-          value="11.8117325473893" />
-        <inertia
-          ixx="0.130576626113656"
-          ixy="1.47971062390579E-07"
-          ixz="0.00285071032522239"
-          iyy="0.168919301848653"
-          iyz="1.07757011014447E-08"
-          izz="0.0962622389900477" />
+          xyz="-0.018464208833126 -0.000195506296033456 -0.0723646952949701"
+          rpy="0 0 0" />
+        <mass
+          value="12.0541385419141" />
+        <inertia
+          ixx="0.130893948352818"
+          ixy="1.47965924737133E-07"
+          ixz="0.00285618491751913"
+          iyy="0.169117950284711"
+          iyz="1.06888893231102E-08"
+          izz="0.0966884532709962" />
       </inertial>
       <visual>
@@ -53,15 +53,15 @@
       <inertial>
         <origin
-          xyz="-2.43019668694222E-06 1.85668461649691E-06 -0.0204728433099643"
-          rpy="0 0 0" />
-        <mass
-          value="0.516905713246417" />
-        <inertia
-          ixx="0.00125613924285597"
-          ixy="2.11747326433519E-09"
-          ixz="2.64299917067243E-08"
-          iyy="0.00125611448213454"
-          iyz="-1.32101831494911E-08"
-          izz="0.00238429646215864" />
+          xyz="-2.43019676260392E-06 1.85668456631483E-06 -0.0204728433099746"
+          rpy="0 0 0" />
+        <mass
+          value="0.516905713246954" />
+        <inertia
+          ixx="0.00125613924285612"
+          ixy="2.1174733006548E-09"
+          ixz="2.64299916603079E-08"
+          iyy="0.00125611448213455"
+          iyz="-1.32101831365386E-08"
+          izz="0.00238429646215876" />
       </inertial>
       <visual>
@@ -107,15 +107,15 @@
       <inertial>
         <origin
-          xyz="3.05776156006576E-06 -3.77816526953012E-08 -0.0204728432555836"
-          rpy="0 0 0" />
-        <mass
-          value="0.516905716540766" />
-        <inertia
-          ixx="0.00125612706197731"
-          ixy="1.24388995856856E-08"
-          ixz="-2.91071422970173E-08"
-          iyy="0.00125612402313693"
-          iyz="-5.16913670862521E-09"
-          izz="0.00238429647597481" />
+          xyz="2.85640525243824E-06 -1.09314890128775E-06 -0.0204728433961597"
+          rpy="0 0 0" />
+        <mass
+          value="0.516905727689722" />
+        <inertia
+          ixx="0.00125613610911781"
+          ixy="8.4818262767786E-09"
+          ixz="-2.90903323912155E-08"
+          iyy="0.00125611767861874"
+          iyz="5.17697116949332E-09"
+          izz="0.00238429652428576" />
       </inertial>
       <visual>
@@ -161,23 +161,23 @@
       <inertial>
         <origin
-          xyz="-0.00849270707917538 0.0122148476204665 9.91213475813879E-05"
-          rpy="0 0 0" />
-        <mass
-          value="0.16436862013948" />
-        <inertia
-          ixx="0.000134032984026512"
-          ixy="4.88470723909831E-05"
-          ixz="-3.22329844113555E-08"
-          iyy="0.000114249682482447"
-          iyz="4.632156635282E-08"
-          izz="0.000205220433201827" />
-      </inertial>
-      <visual>
-        <origin
-          xyz="0 0 0"
-          rpy="0 0 0" />
-        <geometry>
-          <mesh
-            filename="package://yaseen_differential_robot/meshes/caster_left_wheel_link.STL" />
+          xyz="-0.00344828177734346 0.00928242868483165 1.85395651591813E-06"
+          rpy="0 0 0" />
+        <mass
+          value="0.197708449671213" />
+        <inertia
+          ixx="0.000184587750203838"
+          ixy="3.61745827451164E-05"
+          ixz="-2.65414772968982E-06"
+          iyy="0.000123432389094711"
+          iyz="-1.21984397398693E-08"
+          izz="0.000236144832356576" />
+      </inertial>
+      <visual>
+        <origin
+          xyz="0 0 0"
+          rpy="0 0 0" />
+        <geometry>
+          <mesh
+            filename="package://yaseen_differential_robot/meshes/caster_left_link.STL" />
         </geometry>
         <material
@@ -192,5 +192,5 @@
           rpy="0 0 0" />
         <geometry>
-          <sphere radius="0.0372"/>
+          <sphere radius="0.0382"/>
         </geometry>
       </collision>
@@ -217,23 +217,23 @@
       <inertial>
         <origin
-          xyz="-0.00849270707917676 -0.0122148476204665 -9.91213475806524E-05"
-          rpy="0 0 0" />
-        <mass
-          value="0.16436862013948" />
-        <inertia
-          ixx="0.000134032984026512"
-          ixy="-4.88470723909831E-05"
-          ixz="3.22329844113684E-08"
-          iyy="0.000114249682482447"
-          iyz="4.63215663527944E-08"
-          izz="0.000205220433201827" />
-      </inertial>
-      <visual>
-        <origin
-          xyz="0 0 0"
-          rpy="0 0 0" />
-        <geometry>
-          <mesh
-            filename="package://yaseen_differential_robot/meshes/caster_wheel_right_link.STL" />
+          xyz="-0.00344828177734746 -0.00928242868483198 -1.85395651605691E-06"
+          rpy="0 0 0" />
+        <mass
+          value="0.197708449671213" />
+        <inertia
+          ixx="0.000184587750203838"
+          ixy="-3.61745827451162E-05"
+          ixz="-2.6535293449751E-06"
+          iyy="0.000123432389094711"
+          iyz="-1.21984397393522E-08"
+          izz="0.000236144832356577" />
+      </inertial>
+      <visual>
+        <origin
+          xyz="0 0 0"
+          rpy="0 0 0" />
+        <geometry>
+          <mesh
+            filename="package://yaseen_differential_robot/meshes/caster_right_link.STL" />
         </geometry>
         <material
@@ -248,5 +248,5 @@
           rpy="0 0 0" />
         <geometry>
-          <sphere radius="0.0372"/>
+          <sphere radius="0.0382"/>
         </geometry>
       </collision>
@@ -268,5 +268,5 @@
       <inertial>
         <origin
-          xyz="-0.000565454433324009 -1.49381448554266E-05 -0.021701451940591"
+          xyz="-0.000565454433332224 -1.49381448586311E-05 -0.0217014519405859"
           rpy="0 0 0" />
         <mass
@@ -274,8 +274,8 @@
         <inertia
           ixx="7.88651836105335E-05"
-          ixy="4.84717640920677E-08"
+          ixy="4.8471764092049E-08"
           ixz="2.18479443959808E-06"
           iyy="7.51902914938722E-05"
-          iyz="2.88601572509174E-08"
+          iyz="2.88601572509281E-08"
           izz="0.000109946753058707" />
       </inertial>
@@ -308,5 +308,5 @@
       type="fixed">
       <origin
-        xyz="0.2775 -0.00045 -0.4169"
+        xyz="0.2775 -0.01045 -0.36079"
         rpy="0 0 0" />
       <parent
