Commit message: Add Gazebo simulation support with gz_sim
- Add gz_sim.launch.py for Gazebo simulation
- Add robot_gazebo.xacro with Gazebo-specific plugins
- Add gz_controllers.yaml for simulation controllers
- Add empty.sdf world file
- Update robot.urdf.xacro to support use_gazebo argument
- Update robot_ros2_control.xacro with GazeboSimSystem hardware plugin
- Update CMakeLists.txt to install worlds directory
- Fix base_footprint joint name collision for Gazebo compatibility

File: src/yaseen_differential_robot/urdf/robot.urdf.xacro (robot description, xacro)
@@ -2,7 +2,12 @@
 <robot name="yaseen_differential_robot" xmlns:xacro="http://www.ros.org/wiki/xacro">
   <xacro:arg name="use_mock_hardware" default="true" />
+  <xacro:arg name="use_gazebo" default="false" />
   <xacro:include filename="$(find yaseen_differential_robot)/urdf/robot_description.xacro"/>
   <xacro:include filename="$(find yaseen_differential_robot)/urdf/robot_ros2_control.xacro"/>
+  <xacro:include filename="$(find yaseen_differential_robot)/urdf/robot_gazebo.xacro"/>
   <xacro:yaseen_description/>
-  <xacro:yaseen_ros2_control name="YaseenDiffBot" use_mock_hardware="$(arg use_mock_hardware)"/>
+  <xacro:yaseen_ros2_control name="YaseenDiffBot" use_mock_hardware="$(arg use_mock_hardware)" use_gazebo="$(arg use_gazebo)"/>
+  <xacro:if value="$(arg use_gazebo)">
+    <xacro:yaseen_gazebo_plugins/>
+  </xacro:if>
 </robot>

File: src/yaseen_differential_robot/urdf/robot_description.xacro (robot description, xacro)
@@ -43,5 +43,5 @@
     </collision>
   </link>
-  <joint name="base_footprint" type="fixed">
+  <joint name="base_footprint_joint" type="fixed">
     <origin
       xyz="0 0 0.56206"

File: src/yaseen_differential_robot/urdf/robot_ros2_control.xacro (robot description, xacro)
@@ -1,16 +1,23 @@
 <?xml version="1.0"?>
 <robot xmlns:xacro="http://www.ros.org/wiki/xacro">
-  <xacro:macro name="yaseen_ros2_control" params="name use_mock_hardware">
+  <xacro:macro name="yaseen_ros2_control" params="name use_mock_hardware use_gazebo">
     <ros2_control name="${name}" type="system">
-      <xacro:unless value="${use_mock_hardware}">
+      <xacro:unless value="${use_gazebo}">
+        <xacro:unless value="${use_mock_hardware}">
+          <hardware>
+            <plugin>odrive_ros2_control_plugin/ODriveHardwareInterface</plugin>
+            <param name="can">can0</param>
+          </hardware>
+        </xacro:unless>
+        <xacro:if value="${use_mock_hardware}">
+          <hardware>
+            <plugin>mock_components/GenericSystem</plugin>
+            <param name="calculate_dynamics">true</param>
+          </hardware>
+        </xacro:if>
+      </xacro:unless>
+      <xacro:if value="${use_gazebo}">
         <hardware>
-          <plugin>odrive_ros2_control_plugin/ODriveHardwareInterface</plugin>
-          <param name="can">can0</param>
-        </hardware>
-      </xacro:unless>
-      <xacro:if value="${use_mock_hardware}">
-        <hardware>
-          <plugin>mock_components/GenericSystem</plugin>
-          <param name="calculate_dynamics">true</param>
+          <plugin>gz_ros2_control/GazeboSimSystem</plugin>
         </hardware>
       </xacro:if>

Commit message: finalize nav2 and added realsense depth camera urdf

File: src/yaseen_differential_robot/urdf/robot.urdf.xacro (robot description, xacro)
@@ -6,5 +6,7 @@
   <xacro:include filename="$(find yaseen_differential_robot)/urdf/robot_ros2_control.xacro"/>
   <xacro:include filename="$(find yaseen_differential_robot)/urdf/robot_gazebo.xacro"/>
+  <xacro:include filename="$(find yaseen_differential_robot)/urdf/_d435_depth_camera.xacro"/>
   <xacro:yaseen_description/>
+  <xacro:yaseen_depth_camera parent="base_link" use_nominal_extrinsics="false" add_plug="false" use_mesh="true"/>
   <xacro:yaseen_ros2_control name="YaseenDiffBot" use_mock_hardware="$(arg use_mock_hardware)" use_gazebo="$(arg use_gazebo)"/>
   <xacro:if value="$(arg use_gazebo)">

File: src/yaseen_differential_robot/urdf/robot_description.xacro (robot description, xacro)
@@ -317,4 +317,16 @@
         xyz="0 0 0" />
     </joint>
+    <!-- <link name="camera_link"/>
+    <joint
+      name="camera_joint"
+      type="fixed">
+      <origin
+        xyz="0.225 0.00 -0.06"
+        rpy="0 0 0" />
+      <parent
+        link="base_link" />
+      <child
+        link="camera_link" />
+    </joint> -->
   </xacro:macro>
 </robot>
